File: PiSEU-A-v4-discrete.kicad_pcb (KiCad board)
At the start: 4 copper layers, 100 x 100 mm, 114 parts, among them J1 9-32v DC, J11 Buttons, J12 Conn_01x03_Pin, J13 Outputs, J21 Raspberry_Pi_2x20_SMD_Passthr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, J61 I2C GROVE, J62 I2C GROVE, J63 I2C GROVE, J64 I2C-OUTPUTS, J80 ADO 8-Dose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

Commit message: Add files via upload
Parts:
- C27, C30, C31, C32: footprint Capacitor_SMD:C_0603_1608Metric -> Capacitor_THT:C_Disc_D8.0mm_W2.5mm_P5.00mm
- C33: footprint Capacitor_SMD:C_0805_2012Metric -> Capacitor_THT:C_Disc_D8.0mm_W2.5mm_P5.00mm
- moved C27 5.40 mm to (25.7, 15.4), turned to -90 degrees
- moved C31 4.42 mm to (104.6, 105.8)
- moved C32 4.30 mm to (104.7, 102.2), turned to 90 degrees
- moved C30 3.25 mm to (28.8, 15.4), turned to -90 degrees
- moved C33 2.25 mm to (102.5, 87.4), turned to 0 degrees
- moved R30 0.68 mm to (31.8, 14.1)
- moved C26 0.62 mm to (35.3, 14.4)
- moved R33 0.25 mm to (22.7, 21.7)
Connections:
- net Net-(C80-Pad1) renamed /ToneOut
Routing:
- net /pi-5V: track 237.3 -> 160.9 mm
- net /VDC1: track 17.5 -> 10.1 mm, vias 1 -> 0
- net /VDC: track 24.5 -> 19.4 mm
- net Net-(C33-Pad1): track 26.6 -> 22.7 mm
- net Net-(C33-Pad2): track 7.60 -> 3.87 mm
- net /GND: track 13.6 -> 9.89 mm, vias 11 -> 8
- net Net-(C32-Pad1): track 23.4 -> 25.9 mm
- net /IN_RAW: track 110.3 -> 112.2 mm
- net /VTH: track 21.3 -> 19.5 mm
- net Net-(U22A-Cext): track 8.64 -> 7.15 mm
- net /Pi_OFF: vias 1 -> 2
- net /PI_ON: vias 2 -> 3

Commit message: Add files via upload
Parts:
- C1, C11, C12, C13, C14, C20, C22, C23, C25, C29, C32, C33, C64, C65: footprint Capacitor_THT:C_Disc_D8.0mm_W2.5mm_P5.00mm -> Capacitor_THT:C_Disc_D4.7mm_W2.5mm_P5.00mm
- C2, C21, C28: footprint Capacitor_THT:CP_Radial_D10.0mm_P5.00mm_P7.50mm -> Capacitor_THT:CP_Radial_D6.3mm_P2.50mm
- C26, C31: footprint Capacitor_THT:C_Disc_D8.0mm_W2.5mm_P5.00mm -> Capacitor_THT:C_Disc_D5.0mm_W2.5mm_P2.50mm
- C27, C30: footprint Capacitor_THT:C_Disc_D8.0mm_W2.5mm_P5.00mm -> Capacitor_THT:C_Rect_L7.0mm_W4.5mm_P5.00mm
- C63, C73: footprint Capacitor_THT:C_Disc_D7.5mm_W5.0mm_P10.00mm -> Capacitor_THT:C_Rect_L4.6mm_W3.8mm_P2.50mm_MKS02_FKP02
- C66: footprint Capacitor_THT:CP_Radial_D5.0mm_P2.00mm -> Capacitor_THT:CP_Radial_D6.3mm_P2.50mm
- moved C28 31.0 mm to (21.5, 67.3), turned to -90 degrees
- moved C29 29.5 mm to (16.2, 66.0), turned to -90 degrees
- moved C21 24.1 mm to (43.0, 67.3), turned to -90 degrees
- moved C1 16.1 mm to (26.9, 66.0), turned to -90 degrees
- moved JP80 16.0 mm to (75.2, 78.2), turned to 0 degrees
- moved C22 11.4 mm to (37.7, 71.0), turned to 90 degrees
- moved U80 10.7 mm to (75.5, 70.5), turned to 0 degrees
- moved C2 4.84 mm to (32.3, 67.3), turned to -90 degrees
- moved U21 4.75 mm to (47.2, 25.3)
- moved R30 4.72 mm to (36.5, 14.1)
- moved R34 4.54 mm to (25.5, 30.3)
- moved R31 4.54 mm to (35.5, 27.1)
- moved R32 4.54 mm to (35.4, 30.3)
- moved R35 4.54 mm to (17.8, 27.1)
- moved U22 4.53 mm to (51.3, 20.6)
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Routing:
- net /TXD: track 24.6 -> 44.0 mm
- net -5V: track 36.2 -> 24.1 mm
- net +5V: track 37.4 -> 26.2 mm
- net /500HZ: track 137.3 -> 127.2 mm
- net Net-(U80-B): track 19.1 -> 9.29 mm
- net Net-(JP80-C): track 15.9 -> 24.9 mm, vias 0 -> 2
- net /3v3: track 42.2 -> 50.8 mm, vias 5 -> 4
- net /VDC: track 19.4 -> 27.5 mm
- net Net-(U80-C): track 20.1 -> 13.3 mm
- net Net-(C63-Pad2): track 11.8 -> 5.79 mm
- net /700HZ: track 79.7 -> 73.7 mm
- net Net-(C73-Pad2): track 12.1 -> 6.17 mm
- net /VRef: track 73.9 -> 69.2 mm
- net /VDC1: track 10.1 -> 14.6 mm
- net /GND: track 9.89 -> 13.9 mm, vias 8 -> 10
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Other:
- board text added: "1 2 3 4 5 6 7 8"
- board text added: "9-32 Volt"
- board text added: "GPA0 GPA1 GPA2 GPA3 GPA4 GPA5 GPA6 GPA7"
- board text added: "GPB0 GPB1 GPB2 GPB3 GPB4 GPB5 GPB6 GPB7"
- board text added: "center +"
- board text added: "piSEU-A V.4 DISCRETE"
