File: PiSEU-A-v4-discrete.kicad_sch (KiCad schematic)
At the start: 114 parts, among them J1 9-32v DC, J11 Buttons, J12 Conn_01x03_Pin, J13 Outputs, J21 Raspberry_Pi_2x20_SMD_Passthr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, J61 I2C GROVE, J62 I2C GROVE, J63 I2C GROVE, J64 I2C-OUTPUTS, J80 ADO 8-Dose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

Commit message: Add files via upload
Parts:
- C27, C30, C31, C32: footprint Capacitor_SMD:C_0603_1608Metric -> Capacitor_THT:C_Disc_D8.0mm_W2.5mm_P5.00mm
- C33: footprint Capacitor_SMD:C_0805_2012Metric -> Capacitor_THT:C_Disc_D8.0mm_W2.5mm_P5.00mm
Connections:
- net ToneOut: now reaches C80.1, TR80.8
Other:
- moved on the sheet: C31, C32, C33, C34, D21, D80, H25, H26, J80, JP80, R38, R39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

Commit message: Add files via upload
Parts:
- C1, C11, C12, C13, C14, C20, C22, C23, C25, C29, C32, C64, C65: footprint Capacitor_THT:C_Disc_D8.0mm_W2.5mm_P5.00mm -> Capacitor_THT:C_Disc_D4.7mm_W2.5mm_P5.00mm; PARTREV C1590 -> (none); Reichelt (none) -> KERKO 100N
- C2, C21, C28: footprint Capacitor_THT:CP_Radial_D10.0mm_P5.00mm_P7.50mm -> Capacitor_THT:CP_Radial_D6.3mm_P2.50mm; PARTREV C3338 -> (none); Reichelt (none) -> RAD 105 100/35
- C26, C31: footprint Capacitor_THT:C_Disc_D8.0mm_W2.5mm_P5.00mm -> Capacitor_THT:C_Disc_D5.0mm_W2.5mm_P2.50mm; PARTREV C57112 -> (none); Reichelt (none) -> KERKO 10N
- C27: footprint Capacitor_THT:C_Disc_D8.0mm_W2.5mm_P5.00mm -> Capacitor_THT:C_Rect_L7.0mm_W4.5mm_P5.00mm; PARTREV C1597 -> (none); Reichelt (none) -> C3X7R 150NB50
- C30: footprint Capacitor_THT:C_Disc_D8.0mm_W2.5mm_P5.00mm -> Capacitor_THT:C_Rect_L7.0mm_W4.5mm_P5.00mm; PARTREV C21120 -> (none); Reichelt (none) -> C3Z5U 220NB50
- C33: footprint Capacitor_THT:C_Disc_D8.0mm_W2.5mm_P5.00mm -> Capacitor_THT:C_Disc_D4.7mm_W2.5mm_P5.00mm; PARTREV C1595 -> (none); Reichelt (none) -> KERKO 1,5N
- C61, C62, C71, C72: PARTREV C1864297 -> (none); Reichelt (none) -> --
- C63, C73: footprint Capacitor_THT:C_Disc_D7.5mm_W5.0mm_P10.00mm -> Capacitor_THT:C_Rect_L4.6mm_W3.8mm_P2.50mm_MKS02_FKP02; PARTREV C15849 -> (none); Reichelt (none) -> C3X7R 1U 50
- C66: footprint Capacitor_THT:CP_Radial_D5.0mm_P2.00mm -> Capacitor_THT:CP_Radial_D6.3mm_P2.50mm; PARTREV ESL107M016AC3AA -> (none); Reichelt (none) -> RAD 105 100/35
- D20: PARTREV C7420333 -> (none); Reichelt (none) -> BAT 54S SMD
- D21, D80: PARTREV C81598 -> (none); Reichelt (none) -> 1N 4148
- R1, R17, R18, R19, R20, R38: PARTREV C22978 -> (none); Reichelt (none) -> METALL 3,30K
- R11, R14, R15, R16, R24, R25, R37, R67, R77: PARTREV C21190 -> (none); Reichelt (none) -> METALL 1,00K
- R12, R13, R29, R30, R32, R34, R65: PARTREV C25804 -> (none); Reichelt (none) -> METALL 10,0K
- R21, R22: PARTREV C25803 -> (none); Reichelt (none) -> METALL 100K
- R23, R39: PARTREV C181896 -> (none); Reichelt (none) -> METALL 1,60K
- R26: PARTREV C25600 -> (none); Reichelt (none) -> METALL 47,0K
- R27: PARTREV C22935 -> (none); Reichelt (none) -> METALL 1,00M
- R28, R36: PARTREV C31850 -> (none); Reichelt (none) -> METALL 22,0K
- R31: PARTREV C22967 -> (none); Reichelt (none) -> METALL 27,0K
- R33: PARTREV C25804 -> (none); Reichelt (none) -> METALL 4,70K
- R35: PARTREV C25804 -> (none); Reichelt (none) -> METALL 330K
- R40: PARTREV C23138 -> (none); Reichelt (none) -> METALL 330
- R61, R66: PARTREV C1697097 -> (none); Reichelt (none) -> METALL 3,16K
- R62, R63, R72, R73: PARTREV C7115176 -> (none); Reichelt (none) -> METALL 22,0
- R71, R76: PARTREV C1697049 -> (none); Reichelt (none) -> METALL 2,26K
- R80: PARTREV C8218 -> (none); Reichelt (none) -> METALL 200
- U1: PARTREV PRELIMINARY -> (none); Reichelt (none) -> PRELIMINARY
- U11: Reichelt (none) -> ULN 2803A
- U20: PARTREV C185041 -> (none); Reichelt (none) -> --
- U21: PARTREV C41431766 -> (none); Reichelt (none) -> TLC 393 DIP
- U22: PARTREV C26159250 -> (none); Reichelt (none) -> --
- U23: Reichelt (none) -> MCP23017-E/SO
- U61: PARTREV C2878631 -> (none); Reichelt (none) -> --
- U80: PARTREV C6742 -> (none); Reichelt (none) -> SMD 4053
